File: Hardware/rasp_heltec_lora_hat/rasp_heltec_lora_hat/rasp_heltec_lora_hat.kicad_pcb (KiCad board)
At the start: 2 copper layers, 81.3 x 56 mm, 19 parts, among them J1 Conn_I2C_1, J2 Conn_I2C_2, J3 - DAC CONN_DAC2, J4 - ALIMENTACAO Conn_Alim, J5 - ADC1 Con_ADC1, P1 Conn_02x20_Odd_Even, U1 Heltec_Wifi_LoRa_V1

Commit message: Atualizações de hardware:
- Atualizada placa para uso com versão 2 do Heltec LoRa
- Adicionado diodo 1N5819 para permitir funcionamento e programação simultaneos
- Invertidos os conectores I2C para comportar módulos pequenos (exemplo: BMP180) conectaos diretamente na placa
Parts:
- removed Antena LoRa: MountingHole_6.5mm, MountingHole:MountingHole_6.5mm
- removed JP3 - ALIM HELTEC: JMP_ALIM_HELTEC, Connector_PinHeader_2.54mm:PinHeader_1x02_P2.54mm_Vertical
- added ANTENNA (SMA): MountingHole_6mm, MountingHole:MountingHole_6mm, F.Cu at (193.1, 105.0)
- added D2: 1N5819, Diode_THT:D_DO-41_SOD81_P10.16mm_Horizontal, F.Cu at (262.5, 113.4)
- added JP3: JMP_ALIM_HELTEC, Connector_PinHeader_2.54mm:PinHeader_1x02_P2.54mm_Vertical, F.Cu at (262.5, 122.1)
- added REF**: OSHW-Logo2_7.3x6mm_SilkScreen, Symbol:OSHW-Logo2_7.3x6mm_SilkScreen, F.Cu at (202.0, 110.1)
- J3: renamed from J3 - DAC
- J4: renamed from J4 - ALIMENTACAO
- J5: renamed from J5 - ADC1
- JP1: renamed from JP1 - SDA
- JP2: renamed from JP2 - SCL
- MK1, MK2, MK3, MK4: renamed from  
- U1: value Heltec_Wifi_LoRa_V1 -> Heltec_Wifi_LoRa_V2; footprint heltec_wifi_lora_v1:Heltec_WiFi_LoRa_V1 -> heltec_wifi_lora_V2:Heltec_WiFi_LoRa_V2
- moved J2 8.13 mm to (222.9, 131.5), turned to 270 degrees
- moved J1 8.13 mm to (222.9, 136.5), turned to 270 degrees
- moved U1 1.05 mm to (232.5, 114.7)
Connections:
- U1 pad 3: Net-(U1-Pad3) -> VEXT_HELTEC
- U1 pad 34: Net-(U1-Pad3) -> Net-(U1-Pad34)
- U1 pad 35: Net-(JP3-Pad1) -> Net-(U1-Pad34)
- U1 pad 4: GND -> VEXT_HELTEC
Routing:
- net Net-(U1-Pad3): track 24.0 -> 0.00 mm
- net +3V3: track 88.6 -> 72.1 mm
- net GND: track 30.1 -> 44.3 mm
- net Net-(JP3-Pad1): track 32.5 -> 24.9 mm
- net Net-(D2-Pad1): track 0.00 -> 6.10 mm
- net +5V: track 125.8 -> 128.4 mm
- net VEXT_HELTEC: track 0.00 -> 2.54 mm
- net Net-(U1-Pad34): track 0.00 -> 2.48 mm
- net (no net): track 0.00 -> 1.52 mm
- net ADC1_CH_0: track 37.5 -> 38.9 mm
- net ADC1_CH_1: track 40.2 -> 41.6 mm
- net HELTEC_RX: track 7.42 -> 6.30 mm
- net ADC1_CH_2: track 40.6 -> 41.6 mm
- net DAC_OUTPUT: track 33.7 -> 34.5 mm
- net HELTEC_TX: track 18.2 -> 17.5 mm
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Other:
- board text added: "470R"
- board text added: "Heltec LoRa V2"
- board text added: "I²C SDA SCL GND 3V3"
- board text added: "V2"
- board text removed: "***ATENÇÃO *** NÃO PROGRAMAR O HELTEC COM ELE PLUGADO AQUI!"
- board text removed: "I²C 3V3 GND SCL SDA"
